File: power-output/Electrical/power-output.kicad_pcb (KiCad board)
At the start: 2 copper layers, 26 x 30 mm, 27 parts, among them P1 USB_C_Plug_USB2.0, U1 AP2112K-3.3, U2 FUSB302BMPX, U3 LM78L05_SO8, U4 ESP8266EX, U5 CP2102N-Axx-xQFN28

Commit message: Cleared Up power-output project
Parts:
- added C2: 10uF, Capacitor_SMD:C_0201_0603Metric, B.Cu at (140.1, 140.3)
- added J1: Conn_01x02_Socket, Connector_PinSocket_2.54mm:PinSocket_1x02_P2.54mm_Horizontal, F.Cu at (133.5, 145.9)
- C3, R2: moved to B.Cu
- moved R2 6.97 mm to (140.4, 141.5)
- moved U4 6.61 mm to (144.5, 149.7)
- moved C3 5.85 mm to (139.3, 141.7), turned to 90 degrees
- moved C4 1.77 mm to (144.0, 141.5)
Routing:
- net /VCONN: track 48.4 -> 22.1 mm
- net GND: track 119.2 -> 132.8 mm
- net VBUS: track 39.3 -> 47.3 mm
- net /SDA: track 18.3 -> 25.3 mm, vias 2 -> 4
- net /SCL: track 13.3 -> 6.83 mm, vias 2 -> 1
- net /RXD: track 9.09 -> 15.0 mm, vias 2 -> 1
- net /INT: track 28.9 -> 25.1 mm
- net +3.3V: track 80.5 -> 84.3 mm, vias 7 -> 6
- net /TXD: track 11.8 -> 13.1 mm, vias 0 -> 2

Commit message: Cleared power-output project
Parts:
- removed the C5 at (144.8, 134.1)
- removed the C6 at (145.7, 130.7)
- C1, C2: value 10uF -> 1uF
- C9: value 33uF -> 0.33uF
Routing:
- net /VCONN: track 22.1 -> 58.1 mm
- net +3.3V: track 84.3 -> 74.0 mm
- net /SCL: track 6.83 -> 12.7 mm, vias 1 -> 2
- net /CC2: track 3.30 -> 0.00 mm
- net GND: track 132.8 -> 130.4 mm
- net /INT: track 25.1 -> 23.4 mm, vias 3 -> 2
- net VBUS: track 47.3 -> 48.4 mm
- net /RXD: track 15.0 -> 14.3 mm, vias 1 -> 0
