File: CAN-UART/CAN-UART.kicad_pcb (KiCad board)
At the start: 2 copper layers, 26 x 30 mm, 18 parts, among them J1 Conn_01x06, P1 USB_C_Plug_USB2.0, U1 AP2112K-3.3, U2 SN65HVD230, U3 ESP32-C3, U4 AT45DB161D-SU

Commit message: Updated PCB
Parts:
- removed U3: ESP32-C3, Package_DFN_QFN:QFN-32-1EP_5x5mm_P0.5mm_EP3.45x3.45mm
- removed U4: AT45DB161D-SU, Package_SO:SOIC-8_5.275x5.275mm_P1.27mm
- added J2: Screw_Terminal_01x02, Connector_PinHeader_2.54mm:PinHeader_1x02_P2.54mm_Horizontal, F.Cu at (175.3, 155.4)
- added U5: ESP32-C3-MINI-1, Espressif:ESP32-C3-MINI-1U, F.Cu at (141.3, 137.6)
- J1: value Conn_01x06 -> Conn_01x04; footprint Connector_PinSocket_2.00mm:PinSocket_1x06_P2.00mm_Horizontal -> Connector_PinSocket_2.54mm:PinSocket_1x04_P2.54mm_Horizontal
- moved H1 25.0 mm to (151.1, 135.9)
- moved U2 20.1 mm to (130.8, 136.5), turned to -90 degrees
- moved H3 11.4 mm to (129.5, 144.8)
- moved H2 6.60 mm to (151.1, 148.6)
- moved R1 3.75 mm to (133.8, 130.2)
- moved J1 1.04 mm to (129.5, 154.3)
Routing:
- net GND: track 81.4 -> 115.3 mm, vias 5 -> 2
- net +3.3V: track 31.1 -> 0.00 mm
- net /CS: track 18.7 -> 0.00 mm
- net /CAN_TX: track 7.38 -> 24.2 mm, vias 2 -> 0
- net CAN_H: track 16.7 -> 0.00 mm
- net /D-: track 27.3 -> 44.0 mm, vias 0 -> 2
- net /CAN_RX: track 13.0 -> 27.8 mm, vias 2 -> 0
- net /CLK: track 14.8 -> 0.00 mm
- net CAN_L: track 13.8 -> 0.00 mm
- net /MISO: track 11.4 -> 0.00 mm, vias 2 -> 0
- net /RXD: track 15.2 -> 26.4 mm
- net /MOSI: track 10.8 -> 0.00 mm
- net VBUS: track 56.0 -> 66.6 mm, vias 1 -> 2
- net /D+: track 26.2 -> 35.4 mm, vias 0 -> 2
- net /TXD: track 19.3 -> 27.6 mm
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
Commit message: Updated PCB
Parts:
- removed H3: MountingHole, MountingHole:MountingHole_2.2mm_M2
- added Q1: BSS214NW, Package_TO_SOT_SMD:SOT-323_SC-70, F.Cu at (131.4, 142.9)
- added Q2: BSS214NW, Package_TO_SOT_SMD:SOT-323_SC-70, F.Cu at (128.6, 142.7)
- added R2: 60R, Resistor_SMD:R_0402_1005Metric_Pad0.72x0.64mm_HandSolder, F.Cu at (131.5, 145.3)
- added R3: 60R, Resistor_SMD:R_0402_1005Metric_Pad0.72x0.64mm_HandSolder, F.Cu at (128.8, 145.3)
- moved J2 30.7 mm to (144.8, 151.8), turned to -90 degrees
- moved H1 22.5 mm to (129.3, 130.6)
- moved J1 5.09 mm to (129.2, 149.3)
- moved U2 0.90 mm to (130.2, 137.2)
- moved H2 0.57 mm to (151.4, 148.1)
Connections:
- U5 pad 19: unconnected-(U5-GPIO5/ADC2_CH0-Pad19) -> /TERM
Routing:
- net /TERM: track 0.00 -> 27.3 mm, vias 0 -> 2
- net CAN_L: track 0.00 -> 27.2 mm
- net CAN_H: track 0.00 -> 22.0 mm
- net /D-: track 44.0 -> 22.6 mm, vias 2 -> 0
- net VBUS: track 66.6 -> 51.2 mm
- net GND: track 115.3 -> 101.0 mm
- net /D+: track 35.4 -> 22.0 mm, vias 2 -> 0
- net /RXD: track 26.4 -> 18.6 mm
- net /TXD: track 27.6 -> 20.3 mm
- net /CAN_RX: track 27.8 -> 30.5 mm
- net /SDA: track 0.00 -> 1.69 mm, vias 0 -> 1
- net /CAN_TX: track 24.2 -> 25.7 mm
- net /SCL: track 0.00 -> 1.43 mm, vias 0 -> 1
- net +3V3: track 28.2 -> 29.6 mm

Commit message: Updated PCB
Routing:
- net GND: track 101.0 -> 145.1 mm, vias 2 -> 5
- net CAN_L: track 27.2 -> 30.7 mm, vias 0 -> 2
