File: CAN/CAN.kicad_pcb (KiCad board)
At the start: 2 copper layers, 26 x 30 mm, 21 parts, among them J1 Conn_01x04, J2 Screw_Terminal_01x02, P1 USB_C_Plug_USB2.0, Q1 BSS214NW, Q2 BSS214NW, U1 AP2112K-3.3, U2 SN65HVD230, U5 ESP32-C3-MINI-1

Commit message: Updated PCB
Parts:
- removed J2: Screw_Terminal_01x02, Connector_PinHeader_2.54mm:PinHeader_1x02_P2.54mm_Horizontal
- added C10: 0.1uF, Capacitor_SMD:C_0201_0603Metric_Pad0.64x0.40mm_HandSolder, F.Cu at (130.5, 148.1)
- added C11: 0.33uF, Capacitor_SMD:C_0201_0603Metric_Pad0.64x0.40mm_HandSolder, F.Cu at (128.0, 150.4)
- added C12: 0.1uF, Capacitor_SMD:C_0201_0603Metric_Pad0.64x0.40mm_HandSolder, B.Cu at (145.7, 139.4)
- added C13: 0.1uF, Capacitor_SMD:C_0201_0603Metric_Pad0.64x0.40mm_HandSolder, B.Cu at (151.2, 142.0)
- added C5: 1uF, Capacitor_SMD:C_0201_0603Metric_Pad0.64x0.40mm_HandSolder, F.Cu at (149.6, 133.3)
- added C6: 0.1uF, Capacitor_SMD:C_0201_0603Metric_Pad0.64x0.40mm_HandSolder, F.Cu at (149.6, 134.1)
- added C7: 470pF, Capacitor_SMD:C_0201_0603Metric_Pad0.64x0.40mm_HandSolder, F.Cu at (128.0, 148.8)
- added C8: 0.33uF, Capacitor_SMD:C_0201_0603Metric_Pad0.64x0.40mm_HandSolder, B.Cu at (145.7, 137.6)
- added C9: 1uF, Capacitor_SMD:C_0201_0603Metric_Pad0.64x0.40mm_HandSolder, F.Cu at (130.4, 147.3)
- added R4: 4.7k, Resistor_SMD:R_0201_0603Metric, F.Cu at (143.7, 144.8)
- added R5: 4.7k, Resistor_SMD:R_0201_0603Metric, F.Cu at (142.7, 144.9)
- added R6: 4.7k, Resistor_SMD:R_0201_0603Metric, F.Cu at (152.1, 131.1)
- added U3: FUSB302BMPX, Package_DFN_QFN:WQFN-14-1EP_2.5x2.5mm_P0.5mm_EP1.45x1.45mm, F.Cu at (130.8, 150.4)
- added U4: LM78L05_SO8, Package_SO:SOIC-8_3.9x4.9mm_P1.27mm, B.Cu at (130.2, 137.2)
- added U6: LM78L12_SO8, Package_SO:SOIC-8_3.9x4.9mm_P1.27mm, B.Cu at (149.7, 137.3)
- J1: value Conn_01x04 -> Screw_Terminal_01x04; footprint Connector_PinSocket_2.54mm:PinSocket_1x04_P2.54mm_Horizontal -> Connector_PinHeader_2.54mm:PinHeader_1x04_P2.54mm_Horizontal
- moved J1 19.4 mm to (148.3, 152.6), turned to -90 degrees
Connections:
- net Net-(P1-CC) renamed /CC
- C1 pad 1: VBUS -> +5V
- J1 pad 1: VBUS -> +12V
- J1 pad 2: /TXD -> CAN_H
- J1 pad 3: /RXD -> CAN_L
- P1 pad B5: unconnected-(P1-VCONN-PadB5) -> /VCONN
- U1 pad 1: VBUS -> +5V
- U1 pad 3: VBUS -> +5V
- U5 pad 12: unconnected-(U5-GPIO0/ADC1_CH0/XTAL_32K_P-Pad12) -> /INT
- U5 pad 16: /NPXL -> unconnected-(U5-GPIO10-Pad16)
Routing:
- net +5V: track 0.00 -> 88.2 mm, vias 0 -> 5
- net /VCONN: track 0.00 -> 85.8 mm, vias 0 -> 1
- net /INT: track 0.00 -> 61.4 mm, vias 0 -> 3
- net GND: track 145.1 -> 205.6 mm, vias 5 -> 7
- net +3V3: track 29.6 -> 64.9 mm, vias 2 -> 3
- net /CC: track 6.40 -> 40.5 mm, vias 0 -> 5
- net +3.3V: track 0.00 -> 29.7 mm, vias 0 -> 2
- net /SCL: track 1.43 -> 25.3 mm, vias 1 -> 2
- net /SDA: track 1.69 -> 25.3 mm, vias 1 -> 2
- net VBUS: track 51.2 -> 74.1 mm
- net /TXD: track 20.4 -> 0.00 mm, vias 1 -> 0
- net /RXD: track 18.6 -> 0.00 mm, vias 1 -> 0
- net +12V: track 0.00 -> 14.4 mm, vias 0 -> 1
- net /TERM: track 27.3 -> 17.9 mm
- net CAN_L: track 30.7 -> 24.5 mm, vias 2 -> 3
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