File: CAN/CAN.kicad_pcb (KiCad board)
At the start: 2 copper layers, 26 x 30 mm, 18 parts, among them J1 Conn_01x04, J2 Screw_Terminal_01x02, P1 USB_C_Plug_USB2.0, U1 AP2112K-3.3, U2 SN65HVD230, U5 ESP32-C3-MINI-1

Commit message: Updated PCB
Parts:
- removed J1: Conn_01x04, Connector_PinSocket_2.54mm:PinSocket_1x04_P2.54mm_Horizontal
- removed J2: Screw_Terminal_01x02, Connector_PinHeader_2.54mm:PinHeader_1x02_P2.54mm_Horizontal
- added J3: Screw_Terminal_01x04, Connector_PinHeader_2.54mm:PinHeader_1x04_P2.54mm_Horizontal, F.Cu at (71.9, 111.8)
- added Q1: BSS214NW, Package_TO_SOT_SMD:SOT-323_SC-70, F.Cu at (81.3, 108.0)
- added Q2: BSS214NW, Package_TO_SOT_SMD:SOT-323_SC-70, F.Cu at (81.3, 110.9)
- added R2: 60R, Resistor_SMD:R_0402_1005Metric_Pad0.72x0.64mm_HandSolder, F.Cu at (81.0, 105.9)
- added R3: 60R, Resistor_SMD:R_0402_1005Metric_Pad0.72x0.64mm_HandSolder, F.Cu at (80.9, 112.8)
- moved TP1 76.5 mm to (69.5, 87.4)
- moved TP2 76.5 mm to (69.5, 87.4)
- moved U5 76.5 mm to (76.5, 96.9)
- moved C1 76.5 mm to (81.8, 89.2)
- moved C2 76.5 mm to (84.8, 90.4)
- moved C3 76.5 mm to (84.8, 91.2)
- moved C4 76.5 mm to (84.8, 92.0)
- moved H1 76.5 mm to (86.4, 95.3)
- moved H2 76.5 mm to (86.4, 108.0)
- moved H3 76.5 mm to (64.8, 104.2)
- moved P1 76.5 mm to (75.2, 88.4)
- moved R1 76.5 mm to (69.0, 89.5)
- moved TP3 76.5 mm to (80.9, 87.4)
- moved TP4 76.5 mm to (80.9, 87.4)
- moved U1 76.5 mm to (85.0, 88.3)
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Connections:
- U5 pad 16: /NPXL -> unconnected-(U5-GPIO10-Pad16)
- U5 pad 19: unconnected-(U5-GPIO5/ADC2_CH0-Pad19) -> /TERM
- U5 pad 20: /SCL -> unconnected-(U5-GPIO6-Pad20)
- U5 pad 21: /SDA -> unconnected-(U5-GPIO7-Pad21)
Routing:
- net CAN_H: track 0.00 -> 38.3 mm
- net CAN_L: track 0.00 -> 33.8 mm
- net /TXD: track 27.6 -> 0.00 mm, vias 1 -> 0
- net /RXD: track 26.4 -> 0.00 mm, vias 1 -> 0
- net /TERM: track 0.00 -> 11.7 mm, vias 0 -> 2
- net GND: track 115.3 -> 123.8 mm
- net /D-: track 44.0 -> 38.1 mm
