File: uart/Electrical/uart.kicad_pcb (KiCad board)
At the start: 2 copper layers, 26 x 30 mm, 22 parts, among them J1 Conn_01x06, P1 USB_C_Plug_USB2.0, U1 AP2112K-3.3, U2 FT232RL

Commit message: Updated uart PCB
Connections:
- D1 pad 2: a4 -> Net-(D1-A)
Routing:
- net /VDDIO: track 0.00 -> 25.4 mm, vias 0 -> 3
Changed lines of the file:
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@@
   (net 31 "/D+")
   (net 32 "/D-")
+  (net 33 "Net-(D1-A)")
   (footprint "Expansion_Card:USB_C_Plug_Molex_105444" locked (layer "F.Cu")
     (at 159.327793 83.262363)
@@
       (net 3 "VBUS") (pinfunction "K") (pintype "passive"))
     (pad "2" smd roundrect (at 0.32 0) (size 0.46 0.4) (layers "F.Cu" "F.Mask") (roundrect_rratio 0.25)
-      (net 30 "a4") (pinfunction "A") (pintype "passive"))
+      (net 33 "Net-(D1-A)") (pinfunction "A") (pintype "passive"))
     (model "${KICAD6_3DMODEL_DIR}/Diode_SMD.3dshapes/D_0201_0603Metric.wrl"
       (offset (xyz 0 0 0))
@@
   (via (at 167.132 106.68) (size 0.8) (drill 0.4) (layers "F.Cu" "B.Cu") (net 3))
   (via (at 163.068 87.376) (size 0.8) (drill 0.4) (layers "F.Cu" "B.Cu") (net 3))
-  (segment (start 167.132 91.44) (end 167.132 106.68) (width 0.2) (layer "B.Cu") (net 3))
-  (segment (start 163.068 87.376) (end 167.132 91.44) (width 0.2) (layer "B.Cu") (net 3))
+  (segment (start 165.862 90.17) (end 165.862 105.41) (width 0.2) (layer "B.Cu") (net 3))
+  (segment (start 163.068 87.376) (end 165.862 90.17) (width 0.2) (layer "B.Cu") (net 3))
+  (segment (start 165.862 105.41) (end 167.132 106.68) (width 0.2) (layer "B.Cu") (net 3))
   (segment (start 148.209 84.455) (end 148.855 84.455) (width 0.2) (layer "F.Cu") (net 8))
   (segment (start 162.985 94.32) (end 164.374001 94.32) (width 0.2) (layer "F.Cu") (net 8))
@@
   (segment (start 153.924 100.044) (end 153.924 96.012) (width 0.2) (layer "B.Cu") (net 18))
   (segment (start 156.75 102.87) (end 153.924 100.044) (width 0.2) (layer "B.Cu") (net 18))
+  (segment (start 152.337822 92.3205) (end 153.588322 91.07) (width 0.2) (layer "F.Cu") (net 19))
+  (segment (start 147.32 107.696) (end 148.59 107.696) (width 0.2) (layer "F.Cu") (net 19))
+  (segment (start 153.588322 91.07) (end 155.785 91.07) (width 0.2) (layer "F.Cu") (net 19))
+  (segment (start 150.876 107.696) (end 151.13 107.696) (width 0.2) (layer "F.Cu") (net 19))
+  (segment (start 152.333145 92.3205) (end 152.337822 92.3205) (width 0.2) (layer "F.Cu") (net 19))
+  (segment (start 151.13 107.696) (end 151.638 107.188) (width 0.2) (layer "F.Cu") (net 19))
+  (via (at 148.59 107.696) (size 0.8) (drill 0.4) (layers "F.Cu" "B.Cu") (net 19))
+  (via (at 151.638 107.188) (size 0.8) (drill 0.4) (layers "F.Cu" "B.Cu") (net 19))
+  (via (at 152.333145 92.3205) (size 0.8) (drill 0.4) (layers "F.Cu" "B.Cu") (net 19))
+  (segment (start 148.59 107.696) (end 151.13 107.696) (width 0.2) (layer "B.Cu") (net 19))
+  (segment (start 150.684 93.969645) (end 150.684 97.935372) (width 0.2) (layer "B.Cu") (net 19))
+  (segment (start 152.333145 92.3205) (end 150.684 93.969645) (width 0.2) (layer "B.Cu") (net 19))
+  (segment (start 151.13 107.696) (end 151.638 107.188) (width 0.2) (layer "B.Cu") (net 19))
+  (segment (start 151.13 98.381372) (end 151.13 106.68) (width 0.2) (layer "B.Cu") (net 19))
+  (segment (start 150.684 97.935372) (end 151.13 98.381372) (width 0.2) (layer "B.Cu") (net 19))
+  (segment (start 151.13 106.68) (end 151.638 107.188) (width 0.2) (layer "B.Cu") (net 19))
   (segment (start 158.077793 85.386207) (end 157.612 85.852) (width 0.2) (layer "F.Cu") (net 30))
   (segment (start 158.077793 85.386207) (end 158.077793 83.302363) (width 0.2) (layer "F.Cu") (net 30))

Commit message: Updated UART PCB
Parts:
- removed D3, D4: LED, LED_SMD:LED_0201_0603Metric
- removed R3, R4: 1.5k, Resistor_SMD:R_0201_0603Metric
- C1, C2, C3, C4: footprint Capacitor_SMD:C_0805_2012Metric -> Capacitor_SMD:C_0603_1608Metric_Pad1.08x0.95mm_HandSolder
- D1: footprint Diode_SMD:D_0201_0603Metric -> Diode_SMD:D_0603_1608Metric_Pad1.05x0.95mm_HandSolder
- D2: footprint LED_SMD:LED_0201_0603Metric -> LED_SMD:LED_0603_1608Metric_Pad1.05x0.95mm_HandSolder
- J1: footprint Connector_PinHeader_2.00mm:PinHeader_1x06_P2.00mm_Horizontal -> Connector_PinSocket_2.54mm:PinSocket_1x06_P2.54mm_Horizontal
- R1, R2: footprint Resistor_SMD:R_0201_0603Metric -> Resistor_SMD:R_0603_1608Metric_Pad0.98x0.95mm_HandSolder
- moved R2 19.5 mm to (150.3, 106.1)
- moved D2 19.4 mm to (150.3, 109.5)
- moved J1 11.9 mm to (153.0, 101.1), turned to 90 degrees
- moved R1 9.18 mm to (153.7, 87.5), turned to 180 degrees
- moved C4 6.35 mm to (154.3, 93.3)
- moved U2 6.05 mm to (165.0, 91.1), turned to -90 degrees
- moved C3 5.97 mm to (154.3, 91.8)
- moved D1 5.57 mm to (151.7, 85.9)
- moved C1 1.98 mm to (150.0, 87.5), turned to 180 degrees
- moved C2 0.46 mm to (148.3, 85.9)
- moved U1 0.36 mm to (149.7, 83.3)
Connections:
- P1 pad A6: /USB_DP -> /D+
Routing:
- net /CBUS1: track 38.3 -> 0.00 mm
- net /CBUS0: track 37.5 -> 0.00 mm
- net /VDDIO: track 25.4 -> 0.00 mm, vias 3 -> 0
- net VBUS: track 46.8 -> 24.2 mm
- net /RXD: track 15.7 -> 32.5 mm, vias 1 -> 0
- net /D-: track 0.00 -> 16.2 mm, vias 0 -> 2
- net /D+: track 0.00 -> 14.6 mm, vias 0 -> 2
- net GND: track 96.7 -> 83.9 mm, vias 4 -> 5
- net /CTS: track 10.1 -> 21.4 mm
- net /TXD: track 19.1 -> 25.0 mm, vias 1 -> 0
- net /3V3OUT: track 25.6 -> 22.2 mm
- net a4: track 13.3 -> 15.2 mm, vias 1 -> 0
- net +3V3: track 25.3 -> 23.7 mm, vias 2 -> 0
- net /RTS: track 17.8 -> 16.6 mm
- net Net-(D3-A): track 0.98 -> 0.00 mm
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