File: CAN/Electrical/CAN.kicad_sch (KiCad schematic)
At the start: 32 parts, among them J1 Conn_01x05, P1 USB_C_Plug_USB2.0, SW1 Reset, U1 ESP32-C3-MINI-1, U2 AP2112K-3.3, U3 SN65HVD230, U4 FODM217D

Commit message: Updated interactive BOM
Parts:
- H1, H2, TP1, TP2, TP3, TP4, TP5, TP6, TP7, TP8: now left out of the parts list
Changed lines of the file:
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@@
   )
   (symbol (lib_id "Connector:TestPoint") (at 156.21 25.4 0) (unit 1)
-    (in_bom yes) (on_board yes) (dnp no)
+    (in_bom no) (on_board yes) (dnp no)
     (property "Reference" "TP3" (at 157.6832 22.4028 0)
       (effects (font (size 1.27 1.27)) (justify left))
@@
   )
   (symbol (lib_id "Connector:TestPoint") (at 144.78 25.4 0) (unit 1)
-    (in_bom yes) (on_board yes) (dnp no)
+    (in_bom no) (on_board yes) (dnp no)
     (property "Reference" "TP1" (at 146.2532 22.4028 0)
       (effects (font (size 1.27 1.27)) (justify left))
@@
   )
   (symbol (lib_id "Connector:TestPoint") (at 144.78 33.02 0) (unit 1)
-    (in_bom yes) (on_board yes) (dnp no)
+    (in_bom no) (on_board yes) (dnp no)
     (property "Reference" "TP2" (at 146.2532 30.0228 0)
       (effects (font (size 1.27 1.27)) (justify left))
@@
   )
   (symbol (lib_id "Connector:TestPoint") (at 156.21 33.02 0) (unit 1)
-    (in_bom yes) (on_board yes) (dnp no)
+    (in_bom no) (on_board yes) (dnp no)
     (property "Reference" "TP4" (at 157.6832 30.0228 0)
       (effects (font (size 1.27 1.27)) (justify left))
@@
   )
   (symbol (lib_id "Connector:TestPoint") (at 194.31 33.02 0) (unit 1)
-    (in_bom yes) (on_board yes) (dnp no)
+    (in_bom no) (on_board yes) (dnp no)
     (property "Reference" "TP8" (at 195.7832 30.0228 0)
       (effects (font (size 1.27 1.27)) (justify left))
@@
   )
   (symbol (lib_id "Connector:TestPoint") (at 194.31 25.4 0) (unit 1)
-    (in_bom yes) (on_board yes) (dnp no)
+    (in_bom no) (on_board yes) (dnp no)
     (property "Reference" "TP7" (at 195.7832 22.4028 0)
       (effects (font (size 1.27 1.27)) (justify left))
@@
   )
   (symbol (lib_id "Connector:TestPoint") (at 175.26 25.4 0) (unit 1)
-    (in_bom yes) (on_board yes) (dnp no)
+    (in_bom no) (on_board yes) (dnp no)
     (property "Reference" "TP5" (at 176.7332 22.4028 0)
       (effects (font (size 1.27 1.27)) (justify left))
@@
   )
   (symbol (lib_id "Mechanical:MountingHole") (at 209.55 22.86 0) (unit 1)
-    (in_bom yes) (on_board yes) (dnp no)
+    (in_bom no) (on_board yes) (dnp no)
     (property "Reference" "H1" (at 212.09 21.6154 0)
       (effects (font (size 1.27 1.27)) (justify left))
@@
   )
   (symbol (lib_id "Mechanical:MountingHole") (at 209.55 31.75 0) (unit 1)
-    (in_bom yes) (on_board yes) (dnp no)
+    (in_bom no) (on_board yes) (dnp no)
     (property "Reference" "H2" (at 212.09 30.5054 0)
       (effects (font (size 1.27 1.27)) (justify left))
@@
   )
   (symbol (lib_id "Connector:TestPoint") (at 175.26 33.02 0) (unit 1)
-    (in_bom yes) (on_board yes) (dnp no)
+    (in_bom no) (on_board yes) (dnp no)
     (property "Reference" "TP6" (at 176.7332 30.0228 0)
       (effects (font (size 1.27 1.27)) (justify left))

Commit message: Replaced ESP32 Moduole with ESP32-C3
Parts:
- removed C1: 10uF, Capacitor_SMD:C_0805_2012Metric_Pad1.18x1.45mm_HandSolder, symbol Device:C
- removed C2: 1uF, Capacitor_SMD:C_0805_2012Metric_Pad1.18x1.45mm_HandSolder, symbol Device:C
- removed C3: 0.1uF, Capacitor_SMD:C_0805_2012Metric_Pad1.18x1.45mm_HandSolder, symbol Device:C
- removed J1: Conn_01x05, Connector_PinSocket_2.54mm:PinSocket_1x05_P2.54mm_Horizontal, symbol Connector_Generic:Conn_01x05
- removed R1: 10k, Resistor_SMD:R_0805_2012Metric_Pad1.20x1.40mm_HandSolder, symbol Device:R
- removed U1: ESP32-C3-MINI-1, Espressif:ESP32-C3-MINI-1U, symbol Espressif:ESP32-C3-MINI-1
- added C1, C8: 10uF, Capacitor_SMD:C_0805_2012Metric_Pad1.18x1.45mm_HandSolder, symbol Device:C_Small
- added C10, C3: 1uF, Capacitor_SMD:C_0805_2012Metric_Pad1.18x1.45mm_HandSolder, symbol Device:C_Small
- added C11, C12, C14, C15, C2: 0.1uF, Capacitor_SMD:C_0805_2012Metric_Pad1.18x1.45mm_HandSolder, symbol Device:C_Small
- added C4: 1uF, Capacitor_SMD:C_0805_2012Metric_Pad1.18x1.45mm_HandSolder, symbol Device:C
- added C5, C9: TBD, Capacitor_SMD:C_0805_2012Metric_Pad1.18x1.45mm_HandSolder, symbol Device:C_Small
- added C6: 10nF, Capacitor_SMD:C_0805_2012Metric_Pad1.18x1.45mm_HandSolder, symbol Device:C_Small
- added D1: ESD, Diode_SMD:D_0805_2012Metric_Pad1.15x1.40mm_HandSolder, symbol Device:D_TVS_Filled
- added J1: Conn_01x04, Connector_PinSocket_2.54mm:PinSocket_1x04_P2.54mm_Horizontal, symbol Connector_Generic:Conn_01x04
- added L1: 2nH, Inductor_SMD:L_0805_2012Metric_Pad1.15x1.40mm_HandSolder, symbol Device:L_Small
- added R3, R5: 10k, Resistor_SMD:R_0805_2012Metric_Pad1.20x1.40mm_HandSolder, symbol Device:R_Small
- added R4: 0R, Resistor_SMD:R_0805_2012Metric_Pad1.20x1.40mm_HandSolder, symbol Device:R
- added R6: 499R, Resistor_SMD:R_0805_2012Metric_Pad1.20x1.40mm_HandSolder, symbol Device:R_Small
- added U2: ESP32-C3, Package_DFN_QFN:QFN-32-1EP_5x5mm_P0.5mm_EP3.45x3.45mm, symbol Espressif:ESP32-C3
- added Y1: 40MHz, Crystal:Crystal_SMD_TXC_7M-4Pin_3.2x2.5mm, symbol Device:Crystal_GND2
- renumbered C5 to C13, C6 to C16, C4 to C7, D1 to D2, D2 to D3, R2 to R1, R7 to R10, R3 to R2, R4 to R7, R5 to R8, R6 to R9, U2 to U1
Connections:
- net +3.3V: now also C1.1, C11.1, C12.1, C14.1, C2.1, C3.1, C6.1, C8.1, D1.1 (A1), L1.1, R3.1, U2.11 (VDD3P3_RTC), U2.17 (VDD3P3_CPU), U2.31 (VDDA), U2.32 (VDDA)
- net CAN_H: now also J1.2 (Pin_2)
- net CAN_L: now also J1.3 (Pin_3)
- net CAN_RX: now also U2.15 (GPIO9/BOOT)
- net CAN_TX: now also U2.14 (GPIO8)
- net D+: now also U2.26 (GPIO19/USB_D+)
- net D-: now also U2.25 (GPIO18/USB_D-)
- net EN: now also C4.1, R3.2, U2.7 (CHIP_EN)
- net GND: now also C1.2, C10.2, C11.2, C12.2, C14.2, C15.1, C2.2, C3.2, C4.2, C5.2, C6.2, C8.2, C9.2, D1.2 (A2), J1.4 (Pin_4), U2.33 (GND), Y1.2
- net RXD: now also U2.27 (U0RXD/GPIO20)
- net TERM: now also U2.10 (MTDI/GPIO5/ADC2_CH0)
- net TXD: now also R6.2
- net VBUS: now also J1.1 (Pin_1)
- new net: C15.2, L1.2, U2.2 (VDD3P3), U2.3 (VDD3P3)
- new net: C5.1, R4.1, Y1.1
- new net: R6.1, U2.28 (U0TXD/GPIO21)
- new net: R4.2, U2.30 (XTAL_P)
- new net: C9.1, U2.29 (XTAL_N), Y1.3
- new net: R5.2, U2.21 (SPICS0/GPIO14)
- new net VDD_SPI: C10.1, R5.1, U2.18 (VDD_SPI/GPIO11)
- no-connect marks 8 -> 15
Other:
- moved on the sheet: C16, D3, R10, R7, R8, R9, SW1, U3, U4

Commit message: Updated Schematic
Parts:
- removed C1: 10uF, Capacitor_SMD:C_0805_2012Metric_Pad1.18x1.45mm_HandSolder, symbol Device:C_Small
- removed D1: ESD, Diode_SMD:D_0805_2012Metric_Pad1.15x1.40mm_HandSolder, symbol Device:D_TVS_Filled
- added C5: 10uF, Capacitor_SMD:C_0805_2012Metric_Pad1.18x1.45mm_HandSolder, symbol Device:C_Small
- added D2: ESD, Diode_SMD:D_0805_2012Metric_Pad1.15x1.40mm_HandSolder, symbol Device:D_TVS_Filled
- D1: renamed from D2; value D_Schottky -> AVX
- renumbered C7 to C1, C12 to C10, C14 to C11, C15 to C12, C4 to C13, C5 to C14, C9 to C15, C10 to C16, C13 to C2, C16 to C3, C2 to C4, C3 to C6, C6 to C7, C11 to C9, R5 to R10, R10 to R3, R7 to R4, R6 to R5, R3 to R6, R9 to R7, R4 to R9, TP3 to TP2, TP5 to TP3, TP7 to TP4, TP2 to TP5, TP4 to TP6, TP6 to TP7, U3 to U2, U4 to U3, U2 to U4
Connections:
- net +3.3V: now also C5.1, D2.1 (A1)
- net GND: now also C5.2, D2.2 (A2)
Other:
- company: Framework -> Johannes Höllwerth
- title: Expansion Card Template -> CAN - Expansion Card
